Commit message: modify urdf for laser sensor

File: modeldescription/urdf/angelbot.xacro (robot description, xacro)
@@ -6,4 +6,5 @@
  	<!-- Import Rviz colors -->
 	<xacro:include filename="$(find angelbot_sim)/modeldescription/urdf/angelbotmaterial4rviz.xacro"/>
+	<xacro:include filename="$(find angelbot_sim)/modeldescription/urdf/sensors/rplidar_laser.urdf.xacro" />
 	<transmission name="trans_mobile_left">
 		<type>transmission_interface/SimpleTransmission</type>
@@ -82,15 +83,4 @@
 		</inertial>
 	</link>
-	<link name="${robotname}_rplidar">
-		<collision>
-			<geometry>
-				<mesh filename="package://angelbot_sim/modeldescription/mesh/angel_rplidar.STL"></mesh></geometry></collision>
-		<visual>
-			<geometry>
-				<mesh filename="package://angelbot_sim/modeldescription/mesh/angel_rplidar.STL"></mesh></geometry>
-			<material name="red"></material></visual>
-		<inertial>
-			<mass value="0.20856"></mass>
-			<inertia ixx="0.0001" ixy="0.0" ixz="0.0" iyy="0.0002" iyz="0.0" izz="0.0002"></inertia></inertial></link>
 	<joint name="base2shaft" type="fixed">
 		<parent link="${robotname}_base"/>
@@ -110,7 +100,5 @@
 		<axis xyz="0 1 0"/>
 	</joint>
-	<joint name="base2rplidar" type="fixed">
-		<parent link="${robotname}_base"></parent>
-		<child link="${robotname}_rplidar"></child>
-		<origin xyz="-0.0007 0.00015 0.15949"></origin></joint>
+	<xacro:rplidar_laser name="${robotname}" parent="${robotname}_base" ros_topic="/scan" update_rate="40" min_angle="-1.3962634" max_angle="1.3962634" >
+    </xacro:rplidar_laser>
 </robot>

Commit message: update urdf

File: modeldescription/urdf/angelbot.xacro (robot description, xacro)
@@ -7,4 +7,5 @@
 	<xacro:include filename="$(find angelbot_sim)/modeldescription/urdf/angelbotmaterial4rviz.xacro"/>
 	<xacro:include filename="$(find angelbot_sim)/modeldescription/urdf/sensors/rplidar_laser.urdf.xacro" />
+	<xacro:include filename="$(find angelbot_sim)/modeldescription/urdf/sensors/mpu6050_imu.urdf.xacro" />
 	<transmission name="trans_mobile_left">
 		<type>transmission_interface/SimpleTransmission</type>
@@ -100,5 +101,7 @@
 		<axis xyz="0 1 0"/>
 	</joint>
-	<xacro:rplidar_laser name="${robotname}" parent="${robotname}_base" ros_topic="/scan" update_rate="40" min_angle="-1.3962634" max_angle="1.3962634" >
+	<xacro:rplidar_laser name="${robotname}" parent="${robotname}_base" ros_topic="scan" update_rate="40" min_angle="-1.3962634" max_angle="1.3962634" >
     </xacro:rplidar_laser>
+    <xacro:mpu6050_imu name="${robotname}" parent="${robotname}_base">
+    </xacro:mpu6050_imu>
 </robot>

File: modeldescription/urdf/sensors/rplidar_laser.urdf.xacro (robot description, xacro)
@@ -5,5 +5,6 @@
 			<parent link="${parent}"></parent>
 			<child link="${name}_rplidar"></child>
-			<origin xyz="-0.0007 0.00015 0.15949"></origin>
+			<!--  rotate z axis 180 degree according to the placement on angelbot -->
+			<origin xyz="-0.0007 0.00015 0.15949" rpy="0 0 3.1415"></origin>
 		</joint>
 	  	<link name="${name}_rplidar">
